File: stepper-drivers.sch (KiCad schematic (older format))
At the start: 24 parts, among them P16 SW_DIP, P17 SW_DIP, P18 SW_DIP, P19 SW_DIP, U4 4988, U5 4988, U6 4988, U7 4988

Commit message: rc1 route
Parts:
- C10, C11, C12, C9: symbol CP1 -> fabrikator2mini-mk2-rescue:CP1
- P16, P17, P18, P19: symbol CONN_02X03 -> fabrikator2mini-mk2-rescue:CONN_02X03
- R27, R28, R29, R30, R31, R32, R33, R34, R35, R36, R37, R38: symbol R -> fabrikator2mini-mk2-rescue:R
- U4, U5, U6, U7: symbol 4988 -> custom:4988
Changed lines of the file:
@@
-EESchema Schematic File Version 2
-LIBS:fabrikator2mini-mk2-rescue
-LIBS:power
-LIBS:device
-LIBS:transistors
-LIBS:conn
-LIBS:linear
-LIBS:regul
-LIBS:74xx
-LIBS:cmos4000
-LIBS:adc-dac
-LIBS:memory
-LIBS:xilinx
-LIBS:microcontrollers
-LIBS:dsp
-LIBS:microchip
-LIBS:analog_switches
-LIBS:motorola
-LIBS:texas
-LIBS:intel
-LIBS:audio
-LIBS:interface
-LIBS:digital-audio
-LIBS:philips
-LIBS:display
-LIBS:cypress
-LIBS:siliconi
-LIBS:opto
-LIBS:atmel
-LIBS:contrib
-LIBS:valves
-LIBS:custom
-LIBS:ESD_Protection
+EESchema Schematic File Version 4
 LIBS:fabrikator2mini-mk2-cache
-EELAYER 25 0
+EELAYER 26 0
 EELAYER END
 $Descr A4 11693 8268
@@
 $EndDescr
 $Comp
-L 4988 U4
+L custom:4988 U4
 U 1 1 5A6FCEDD
 P 2550 2250
@@
 $EndComp
 $Comp
-L 4988 U5
+L custom:4988 U5
 U 1 1 5A6FCEE4
 P 5400 2250
@@
 $EndComp
 $Comp
-L 4988 U6
+L custom:4988 U6
 U 1 1 5A6FCEEB
 P 8500 2250
@@
 $EndComp
 $Comp
-L 4988 U7
+L custom:4988 U7
 U 1 1 5A6FCEF2
 P 2700 4850
@@
 $EndComp
 $Comp
-L GND #PWR058
+L power:GND #PWR058
 U 1 1 5A6FCEF9
 P 3250 5100
@@
 $EndComp
 $Comp
-L GND #PWR059
+L power:GND #PWR059
 U 1 1 5A6FCEFF
 P 3250 4500
@@
 $EndComp
 $Comp
-L GND #PWR060
+L power:GND #PWR060
 U 1 1 5A6FCF05
 P 9050 2500
@@
 $EndComp
 $Comp
-L GND #PWR061
+L power:GND #PWR061
 U 1 1 5A6FCF0B
 P 9050 1900
@@
 $EndComp
 $Comp
-L GND #PWR062
+L power:GND #PWR062
 U 1 1 5A6FCF11
 P 5950 2500
@@
 $EndComp
 $Comp
-L GND #PWR063
+L power:GND #PWR063
 U 1 1 5A6FCF17
 P 5950 1900
@@
 $EndComp
 $Comp
-L GND #PWR064
+L power:GND #PWR064
 U 1 1 5A6FCF1D
 P 3100 2500
@@
 $EndComp
 $Comp
-L GND #PWR065
+L power:GND #PWR065
 U 1 1 5A6FCF23
 P 3100 1900
@@
 $EndComp
 $Comp
-L +3.3V #PWR066
+L power:+3.3V #PWR066
 U 1 1 5A6FCF29
 P 3100 2000
@@
 $EndComp
 $Comp
-L +3.3V #PWR067
+L power:+3.3V #PWR067
 U 1 1 5A6FCF2F
 P 5950 2000
@@
 $EndComp
 $Comp
-L +3.3V #PWR068
+L power:+3.3V #PWR068
 U 1 1 5A6FCF35
 P 9050 2000
@@
 $EndComp
 $Comp
-L +3.3V #PWR069
+L power:+3.3V #PWR069
 U 1 1 5A6FCF3B
 P 3250 4600
@@
 Z_2B
 $Comp
-L CONN_02X03 P16
+L fabrikator2mini-mk2-rescue:CONN_02X03 P16
 U 1 1 5A6FCF5B
 P 1650 2100
@@
 $EndComp
 $Comp
-L CONN_02X03 P17
+L fabrikator2mini-mk2-rescue:CONN_02X03 P17
 U 1 1 5A6FCF62
 P 4500 2100
@@
 $EndComp
 $Comp
-L CONN_02X03 P18
+L fabrikator2mini-mk2-rescue:CONN_02X03 P18
 U 1 1 5A6FCF69
 P 7600 2100
@@
 $EndComp
 $Comp
-L CONN_02X03 P19
+L fabrikator2mini-mk2-rescue:CONN_02X03 P19
 U 1 1 5A6FCF70
 P 1800 4700
@@
 $EndComp
 $Comp
-L +3.3V #PWR070
+L power:+3.3V #PWR070
 U 1 1 5A6FCF77
 P 1500 4550
@@
 $EndComp
 $Comp
-L +3.3V #PWR071
+L power:+3.3V #PWR071
 U 1 1 5A6FCF7D
 P 7300 1950
@@
 $EndComp
 $Comp
-L +3.3V #PWR072
+L power:+3.3V #PWR072
 U 1 1 5A6FCF83
 P 4200 1950
@@
 $EndComp
 $Comp
-L +3.3V #PWR073
+L power:+3.3V #PWR073
 U 1 1 5A6FCF89
 P 1350 1950
@@
 $EndComp
 $Comp
-L R R27
+L fabrikator2mini-mk2-rescue:R R27
 U 1 1 5A6FCF8F
 P 2000 1700
@@
 $EndComp
 $Comp
-L R R28
+L fabrikator2mini-mk2-rescue:R R28
 U 1 1 5A6FCF96
 P 4850 1700
@@
 $EndComp
 $Comp
-L R R29
+L fabrikator2mini-mk2-rescue:R R29
 U 1 1 5A6FCF9D
 P 7950 1700
@@
 $EndComp
 $Comp
-L R R36
+L fabrikator2mini-mk2-rescue:R R36
 U 1 1 5A6FCFA4
 P 2150 4300
@@
 $EndComp
 $Comp
-L R R37
+L fabrikator2mini-mk2-rescue:R R37
 U 1 1 5A6FCFAB
 P 1350 4900
@@
 $EndComp
 $Comp
-L R R32
+L fabrikator2mini-mk2-rescue:R R32
 U 1 1 5A6FCFB2
 P 7150 2300
@@
 $EndComp
 $Comp
-L R R31
+L fabrikator2mini-mk2-rescue:R R31
 U 1 1 5A6FCFB9
 P 4050 2300
@@
 $EndComp
 $Comp
-L R R30
+L fabrikator2mini-mk2-rescue:R R30
 U 1 1 5A6FCFC0
 P 1200 2300
@@
 $EndComp
 $Comp
-L +3.3V #PWR074
+L power:+3.3V #PWR074
 U 1 1 5A6FCFC7
 P 2000 1500
@@
 $EndComp
 $Comp
-L +3.3V #PWR075
+L power:+3.3V #PWR075
 U 1 1 5A6FCFCD
 P 4850 1500
@@
 $EndComp
 $Comp
-L +3.3V #PWR076
+L power:+3.3V #PWR076
 U 1 1 5A6FCFD3
 P 7950 1500
@@
 $EndComp
 $Comp
-L +3.3V #PWR077
+L power:+3.3V #PWR077
 U 1 1 5A6FCFD9
 P 2150 4100
@@
 $EndComp
 $Comp
-L GND #PWR078
+L power:GND #PWR078
 U 1 1 5A6FCFDF
 P 1150 4900
@@
 $EndComp
 $Comp
-L GND #PWR079
+L power:GND #PWR079
 U 1 1 5A6FCFE5
 P 6950 2300
@@
 $EndComp
 $Comp
-L GND #PWR080
+L power:GND #PWR080
 U 1 1 5A6FCFEB
 P 3850 2300
@@
 $EndComp
 $Comp
-L GND #PWR081
+L power:GND #PWR081
 U 1 1 5A6FCFF1
 P 1000 2300
@@
 $EndComp
 $Comp
-L VCC #PWR082
+L power:VCC #PWR082
 U 1 1 5A6FCFF7
 P 3100 2600
@@
 $EndComp
 $Comp
-L VCC #PWR083
+L power:VCC #PWR083
 U 1 1 5A6FCFFD
 P 5950 2600
@@
 $EndComp
 $Comp
-L VCC #PWR084
+L power:VCC #PWR084
 U 1 1 5A6FD003
 P 9050 2600
@@
 $EndComp
 $Comp
-L VCC #PWR085
+L power:VCC #PWR085
 U 1 1 5A6FD009
 P 3250 5200
@@
 	4850 1500 4850 1550
 $Comp
-L R R33
+L fabrikator2mini-mk2-rescue:R R33
 U 1 1 5A6FDA23
 P 1200 2400
@@
 $EndComp
 $Comp
-L +3.3V #PWR086
+L power:+3.3V #PWR086
 U 1 1 5A6FDA76
 P 1000 2400
@@
 Connection ~ 2000 2350
 $Comp
-L CP1 C10
+L fabrikator2mini-mk2-rescue:CP1 C10
 U 1 1 5A6FE7C0
 P 5100 4650
@@
 $EndComp
 $Comp
-L CP1 C11
+L fabrikator2mini-mk2-rescue:CP1 C11
 U 1 1 5A6FE7C7
 P 5400 4650
@@
 $EndComp
 $Comp
-L CP1 C12
+L fabrikator2mini-mk2-rescue:CP1 C12
 U 1 1 5A6FE7CE
 P 5700 4650
@@
 $EndComp
 $Comp
-L CP1 C9
+L fabrikator2mini-mk2-rescue:CP1 C9
 U 1 1 5A6FE7D5
 P 4800 4650
@@
 $EndComp
 $Comp
-L GND #PWR087
+L power:GND #PWR087
 U 1 1 5A6FE7DC
 P 5250 4900
@@
 $EndComp
 $Comp
-L VCC #PWR088
+L power:VCC #PWR088
 U 1 1 5A6FE7E2
 P 5250 4400
@@
 Connection ~ 5400 4850
 $Comp
-L R R38
+L fabrikator2mini-mk2-rescue:R R38
 U 1 1 5A7089A4
 P 1350 5000
@@
 $EndComp
 $Comp
-L R R34
+L fabrikator2mini-mk2-rescue:R R34
 U 1 1 5A708A64
 P 4050 2400
@@
 $EndComp
 $Comp
-L R R35
+L fabrikator2mini-mk2-rescue:R R35
 U 1 1 5A708B30
 P 7150 2400
@@
 $EndComp
 $Comp
-L +3.3V #PWR089
+L power:+3.3V #PWR089
 U 1 1 5A708C4C
 P 1150 5000
@@
 $EndComp
 $Comp
-L +3.3V #PWR090
+L power:+3.3V #PWR090
 U 1 1 5A708C9F
 P 3850 2400
@@
 $EndComp
 $Comp
-L +3.3V #PWR091
+L power:+3.3V #PWR091
 U 1 1 5A708DCA
 P 6950 2400

Commit message: fixed symbols after switch to kicad 5
Parts:
- C10, C11, C12, C9: symbol fabrikator2mini-mk2-rescue:CP1 -> Device:CP1
- P16, P17, P18, P19: symbol fabrikator2mini-mk2-rescue:CONN_02X03 -> Connector_Generic:Conn_02x03_Odd_Even
- R27, R28, R29, R30, R31, R32, R33, R34, R35, R36, R37, R38: symbol fabrikator2mini-mk2-rescue:R -> Device:R
Changed lines of the file:
@@
 Z_2B
 $Comp
-L fabrikator2mini-mk2-rescue:CONN_02X03 P16
+L Connector_Generic:Conn_02x03_Odd_Even P16
 U 1 1 5A6FCF5B
-P 1650 2100
-F 0 "P16" H 1650 2300 50  0000 C CNN
-F 1 "SW_DIP" H 1650 1900 50  0000 C CNN
-F 2 "Pin_Headers:Pin_Header_Straight_2x03_Pitch2.54mm" H 1650 900 50  0001 C CNN
-F 3 "" H 1650 900 50  0000 C CNN
-	1    1650 2100
+P 1600 2100
+F 0 "P16" H 1600 2300 50  0000 C CNN
+F 1 "SW_DIP" H 1600 1900 50  0000 C CNN
+F 2 "Pin_Headers:Pin_Header_Straight_2x03_Pitch2.54mm" H 1600 900 50  0001 C CNN
+F 3 "" H 1600 900 50  0000 C CNN
+	1    1600 2100
 	1    0    0    1
 $EndComp
 $Comp
-L fabrikator2mini-mk2-rescue:CONN_02X03 P17
+L Connector_Generic:Conn_02x03_Odd_Even P17
 U 1 1 5A6FCF62
-P 4500 2100
-F 0 "P17" H 4500 2300 50  0000 C CNN
-F 1 "SW_DIP" H 4500 1900 50  0000 C CNN
-F 2 "Pin_Headers:Pin_Header_Straight_2x03_Pitch2.54mm" H 4500 900 50  0001 C CNN
-F 3 "" H 4500 900 50  0000 C CNN
-	1    4500 2100
+P 4450 2100
+F 0 "P17" H 4450 2300 50  0000 C CNN
+F 1 "SW_DIP" H 4450 1900 50  0000 C CNN
+F 2 "Pin_Headers:Pin_Header_Straight_2x03_Pitch2.54mm" H 4450 900 50  0001 C CNN
+F 3 "" H 4450 900 50  0000 C CNN
+	1    4450 2100
 	1    0    0    1
 $EndComp
 $Comp
-L fabrikator2mini-mk2-rescue:CONN_02X03 P18
+L Connector_Generic:Conn_02x03_Odd_Even P18
 U 1 1 5A6FCF69
-P 7600 2100
-F 0 "P18" H 7600 2300 50  0000 C CNN
-F 1 "SW_DIP" H 7600 1900 50  0000 C CNN
-F 2 "Pin_Headers:Pin_Header_Straight_2x03_Pitch2.54mm" H 7600 900 50  0001 C CNN
-F 3 "" H 7600 900 50  0000 C CNN
-	1    7600 2100
+P 7550 2100
+F 0 "P18" H 7550 2300 50  0000 C CNN
+F 1 "SW_DIP" H 7550 1900 50  0000 C CNN
+F 2 "Pin_Headers:Pin_Header_Straight_2x03_Pitch2.54mm" H 7550 900 50  0001 C CNN
+F 3 "" H 7550 900 50  0000 C CNN
+	1    7550 2100
 	1    0    0    1
 $EndComp
 $Comp
-L fabrikator2mini-mk2-rescue:CONN_02X03 P19
+L Connector_Generic:Conn_02x03_Odd_Even P19
 U 1 1 5A6FCF70
-P 1800 4700
-F 0 "P19" H 1800 4900 50  0000 C CNN
-F 1 "SW_DIP" H 1800 4500 50  0000 C CNN
-F 2 "Pin_Headers:Pin_Header_Straight_2x03_Pitch2.54mm" H 1800 3500 50  0001 C CNN
-F 3 "" H 1800 3500 50  0000 C CNN
-	1    1800 4700
+P 1750 4700
+F 0 "P19" H 1750 4900 50  0000 C CNN
+F 1 "SW_DIP" H 1750 4500 50  0000 C CNN
+F 2 "Pin_Headers:Pin_Header_Straight_2x03_Pitch2.54mm" H 1750 3500 50  0001 C CNN
+F 3 "" H 1750 3500 50  0000 C CNN
+	1    1750 4700
 	1    0    0    1
 $EndComp
@@
 $EndComp
 $Comp
-L fabrikator2mini-mk2-rescue:R R27
+L Device:R R27
 U 1 1 5A6FCF8F
 P 2000 1700
@@
 $EndComp
 $Comp
-L fabrikator2mini-mk2-rescue:R R28
+L Device:R R28
 U 1 1 5A6FCF96
 P 4850 1700
@@
 $EndComp
 $Comp
-L fabrikator2mini-mk2-rescue:R R29
+L Device:R R29
 U 1 1 5A6FCF9D
 P 7950 1700
@@
 $EndComp
 $Comp
-L fabrikator2mini-mk2-rescue:R R36
+L Device:R R36
 U 1 1 5A6FCFA4
 P 2150 4300
@@
 $EndComp
 $Comp
-L fabrikator2mini-mk2-rescue:R R37
+L Device:R R37
 U 1 1 5A6FCFAB
 P 1350 4900
@@
 $EndComp
 $Comp
-L fabrikator2mini-mk2-rescue:R R32
+L Device:R R32
 U 1 1 5A6FCFB2
 P 7150 2300
@@
 $EndComp
 $Comp
-L fabrikator2mini-mk2-rescue:R R31
+L Device:R R31
 U 1 1 5A6FCFB9
 P 4050 2300
@@
 $EndComp
 $Comp
-L fabrikator2mini-mk2-rescue:R R30
+L Device:R R30
 U 1 1 5A6FCFC0
 P 1200 2300
@@
 	2050 2600 2000 2600
 Wire Wire Line
-	1950 1900 2050 1900
-Wire Wire Line
-	4800 1900 4900 1900
+	1950 1900 2000 1900
+Wire Wire Line
+	4800 1900 4850 1900
 Wire Wire Line
 	4850 2500 4900 2500
@@
 	8000 2500 7950 2500
 Wire Wire Line
-	7900 1900 8000 1900
-Wire Wire Line
-	2100 4500 2200 4500
+	7900 1900 7950 1900
+Wire Wire Line
+	2100 4500 2150 4500
 Wire Wire Line
 	2150 5100 2200 5100
@@
 	2200 5000 2150 5000
 Wire Wire Line
-	2150 5000 2150 4900
+	2150 5000 2150 4950
 Wire Wire Line
 	2150 4900 2200 4900
@@
 	8000 2400 7950 2400
 Wire Wire Line
-	7950 2400 7950 2300
+	7950 2400 7950 2350
 Wire Wire Line
 	7950 2300 8000 2300
@@
 	4900 2400 4850 2400
 Wire Wire Line
-	4850 2400 4850 2300
+	4850 2400 4850 2350
 Wire Wire Line
 	4850 2300 4900 2300
@@
 	2000 2400 2050 2400
 Wire Wire Line
-	2000 2300 2000 2400
+	2000 2300 2000 2350
 Wire Wire Line
 	2000 2300 2050 2300
@@
 	1500 4800 1550 4800
 Wire Wire Line
-	1500 4550 1500 4800
+	1500 4550 1500 4600
 Wire Wire Line
 	1550 4600 1500 4600
@@
 	2200 4700 2050 4700
 Wire Wire Line
-	2050 4600 2200 4600
-Wire Wire Line
-	7850 2000 8000 2000
+	2050 4600 2100 4600
+Wire Wire Line
+	7850 2000 7900 2000
 Wire Wire Line
 	8000 2100 7850 2100
@@
 	7300 2200 7350 2200
 Wire Wire Line
-	7300 1950 7300 2200
+	7300 1950 7300 2000
 Wire Wire Line
 	7300 2000 7350 2000
@@
 Connection ~ 1350 2100
 Wire Wire Line
-	1900 2000 2050 2000
+	1900 2000 1950 2000
 Wire Wire Line
 	2050 2100 1900 2100
@@
 	1900 2200 2050 2200
 Wire Wire Line
-	4750 2000 4900 2000
+	4750 2000 4800 2000
 Wire Wire Line
 	4900 2100 4750 2100
@@
 	4200 2000 4250 2000
 Wire Wire Line
-	4200 1950 4200 2200
-Wire Wire Line
-	1350 1950 1350 2200
+	4200 1950 4200 2000
+Wire Wire Line
+	1350 1950 1350 2000
 Wire Wire Line
 	1050 2300 1000 2300
@@
 	4850 1500 4850 1550
 $Comp
-L fabrikator2mini-mk2-rescue:R R33
+L Device:R R33
 U 1 1 5A6FDA23
 P 1200 2400
@@
 Connection ~ 2000 2350
 $Comp
-L fabrikator2mini-mk2-rescue:CP1 C10
+L Device:CP1 C10
 U 1 1 5A6FE7C0
 P 5100 4650
@@
 $EndComp
 $Comp
-L fabrikator2mini-mk2-rescue:CP1 C11
+L Device:CP1 C11
 U 1 1 5A6FE7C7
 P 5400 4650
@@
 $EndComp
 $Comp
-L fabrikator2mini-mk2-rescue:CP1 C12
+L Device:CP1 C12
 U 1 1 5A6FE7CE
 P 5700 4650
@@
 $EndComp
 $Comp
-L fabrikator2mini-mk2-rescue:CP1 C9
+L Device:CP1 C9
 U 1 1 5A6FE7D5
 P 4800 4650
@@
 	4800 4500 4800 4450
 Wire Wire Line
-	4800 4450 5700 4450
+	4800 4450 5100 4450
 Wire Wire Line
 	5700 4450 5700 4500
@@
 	4800 4800 4800 4850
 Wire Wire Line
-	4800 4850 5700 4850
+	4800 4850 5100 4850
 Wire Wire Line
 	5700 4850 5700 4800
@@
 Connection ~ 5400 4850
 $Comp
-L fabrikator2mini-mk2-rescue:R R38
+L Device:R R38
 U 1 1 5A7089A4
 P 1350 5000
@@
 $EndComp
 $Comp
-L fabrikator2mini-mk2-rescue:R R34
+L Device:R R34
 U 1 1 5A708A64
 P 4050 2400
@@
 $EndComp
 $Comp
-L fabrikator2mini-mk2-rescue:R R35
+L Device:R R35
 U 1 1 5A708B30
 P 7150 2400
@@
 Text GLabel 3250 5000 2    60   Input ~ 0
 E_2B
+Wire Wire Line
+	1500 4600 1500 4700
+Wire Wire Line
+	1500 4700 1500 4800
+Wire Wire Line
+	7300 2000 7300 2100
+Wire Wire Line
+	7300 2100 7300 2200
+Wire Wire Line
+	4200 2000 4200 2100
+Wire Wire Line
+	1350 2000 1350 2100
+Wire Wire Line
+	1350 2100 1350 2200
+Wire Wire Line
+	4200 2100 4200 2200
+Wire Wire Line
+	2000 1900 2050 1900
+Wire Wire Line
+	4850 1900 4900 1900
+Wire Wire Line
+	1950 2000 2050 2000
+Wire Wire Line
+	4800 2000 4900 2000
+Wire Wire Line
+	7900 2000 8000 2000
+Wire Wire Line
+	7950 1900 8000 1900
+Wire Wire Line
+	2150 4500 2200 4500
+Wire Wire Line
+	2100 4600 2200 4600
+Wire Wire Line
+	2000 2350 2000 2400
+Wire Wire Line
+	5250 4850 5400 4850
+Wire Wire Line
+	5250 4450 5400 4450
+Wire Wire Line
+	5100 4450 5250 4450
+Wire Wire Line
+	5100 4850 5250 4850
+Wire Wire Line
+	5400 4450 5700 4450
+Wire Wire Line
+	5400 4850 5700 4850
+Wire Wire Line
+	4850 2350 4850 2300
+Wire Wire Line
+	7950 2350 7950 2300
+Wire Wire Line
+	2150 4950 2150 4900
 $EndSCHEMATC

Commit message: fixed modules after switch to kicad 5
Parts:
- C10, C11, C12, C9: footprint Capacitors_SMD:CP_Elec_8x10 -> Capacitor_SMD:CP_Elec_8x10
- P16, P17, P18, P19: footprint Pin_Headers:Pin_Header_Straight_2x03_Pitch2.54mm -> Connector_PinHeader_2.54mm:PinHeader_2x03_P2.54mm_Vertical
- R27, R28, R29, R30, R31, R32, R33, R34, R35, R36, R37, R38: footprint Resistors_SMD:R_0805_HandSoldering -> Resistor_SMD:R_0805_2012Metric_Pad1.15x1.40mm_HandSolder
Changed lines of the file:
@@
 F 0 "P16" H 1600 2300 50  0000 C CNN
 F 1 "SW_DIP" H 1600 1900 50  0000 C CNN
-F 2 "Pin_Headers:Pin_Header_Straight_2x03_Pitch2.54mm" H 1600 900 50  0001 C CNN
+F 2 "Connector_PinHeader_2.54mm:PinHeader_2x03_P2.54mm_Vertical" H 1600 900 50  0001 C CNN
 F 3 "" H 1600 900 50  0000 C CNN
 	1    1600 2100
@@
 F 0 "P17" H 4450 2300 50  0000 C CNN
 F 1 "SW_DIP" H 4450 1900 50  0000 C CNN
-F 2 "Pin_Headers:Pin_Header_Straight_2x03_Pitch2.54mm" H 4450 900 50  0001 C CNN
+F 2 "Connector_PinHeader_2.54mm:PinHeader_2x03_P2.54mm_Vertical" H 4450 900 50  0001 C CNN
 F 3 "" H 4450 900 50  0000 C CNN
 	1    4450 2100
@@
 F 0 "P18" H 7550 2300 50  0000 C CNN
 F 1 "SW_DIP" H 7550 1900 50  0000 C CNN
-F 2 "Pin_Headers:Pin_Header_Straight_2x03_Pitch2.54mm" H 7550 900 50  0001 C CNN
+F 2 "Connector_PinHeader_2.54mm:PinHeader_2x03_P2.54mm_Vertical" H 7550 900 50  0001 C CNN
 F 3 "" H 7550 900 50  0000 C CNN
 	1    7550 2100
@@
 F 0 "P19" H 1750 4900 50  0000 C CNN
 F 1 "SW_DIP" H 1750 4500 50  0000 C CNN
-F 2 "Pin_Headers:Pin_Header_Straight_2x03_Pitch2.54mm" H 1750 3500 50  0001 C CNN
+F 2 "Connector_PinHeader_2.54mm:PinHeader_2x03_P2.54mm_Vertical" H 1750 3500 50  0001 C CNN
 F 3 "" H 1750 3500 50  0000 C CNN
 	1    1750 4700
@@
 F 0 "R27" V 2080 1700 50  0000 C CNN
 F 1 "10k" V 2000 1700 50  0000 C CNN
-F 2 "Resistors_SMD:R_0805_HandSoldering" V 1930 1700 50  0001 C CNN
+F 2 "Resistor_SMD:R_0805_2012Metric_Pad1.15x1.40mm_HandSolder" V 1930 1700 50  0001 C CNN
 F 3 "" H 2000 1700 50  0000 C CNN
 	1    2000 1700
@@
 F 0 "R28" V 4930 1700 50  0000 C CNN
 F 1 "10k" V 4850 1700 50  0000 C CNN
-F 2 "Resistors_SMD:R_0805_HandSoldering" V 4780 1700 50  0001 C CNN
+F 2 "Resistor_SMD:R_0805_2012Metric_Pad1.15x1.40mm_HandSolder" V 4780 1700 50  0001 C CNN
 F 3 "" H 4850 1700 50  0000 C CNN
 	1    4850 1700
@@
 F 0 "R29" V 8030 1700 50  0000 C CNN
 F 1 "10k" V 7950 1700 50  0000 C CNN
-F 2 "Resistors_SMD:R_0805_HandSoldering" V 7880 1700 50  0001 C CNN
+F 2 "Resistor_SMD:R_0805_2012Metric_Pad1.15x1.40mm_HandSolder" V 7880 1700 50  0001 C CNN
 F 3 "" H 7950 1700 50  0000 C CNN
 	1    7950 1700
@@
 F 0 "R36" V 2230 4300 50  0000 C CNN
 F 1 "10k" V 2150 4300 50  0000 C CNN
-F 2 "Resistors_SMD:R_0805_HandSoldering" V 2080 4300 50  0001 C CNN
+F 2 "Resistor_SMD:R_0805_2012Metric_Pad1.15x1.40mm_HandSolder" V 2080 4300 50  0001 C CNN
 F 3 "" H 2150 4300 50  0000 C CNN
 	1    2150 4300
@@
 F 0 "R37" V 1430 4900 50  0000 C CNN
 F 1 "10k" V 1350 4900 50  0000 C CNN
-F 2 "Resistors_SMD:R_0805_HandSoldering" V 1280 4900 50  0001 C CNN
+F 2 "Resistor_SMD:R_0805_2012Metric_Pad1.15x1.40mm_HandSolder" V 1280 4900 50  0001 C CNN
 F 3 "" H 1350 4900 50  0000 C CNN
 	1    1350 4900
@@
 F 0 "R32" V 7230 2300 50  0000 C CNN
 F 1 "10k" V 7150 2300 50  0000 C CNN
-F 2 "Resistors_SMD:R_0805_HandSoldering" V 7080 2300 50  0001 C CNN
+F 2 "Resistor_SMD:R_0805_2012Metric_Pad1.15x1.40mm_HandSolder" V 7080 2300 50  0001 C CNN
 F 3 "" H 7150 2300 50  0000 C CNN
 	1    7150 2300
@@
 F 0 "R31" V 4130 2300 50  0000 C CNN
 F 1 "10k" V 4050 2300 50  0000 C CNN
-F 2 "Resistors_SMD:R_0805_HandSoldering" V 3980 2300 50  0001 C CNN
+F 2 "Resistor_SMD:R_0805_2012Metric_Pad1.15x1.40mm_HandSolder" V 3980 2300 50  0001 C CNN
 F 3 "" H 4050 2300 50  0000 C CNN
 	1    4050 2300
@@
 F 0 "R30" V 1280 2300 50  0000 C CNN
 F 1 "10k" V 1200 2300 50  0000 C CNN
-F 2 "Resistors_SMD:R_0805_HandSoldering" V 1130 2300 50  0001 C CNN
+F 2 "Resistor_SMD:R_0805_2012Metric_Pad1.15x1.40mm_HandSolder" V 1130 2300 50  0001 C CNN
 F 3 "" H 1200 2300 50  0000 C CNN
 	1    1200 2300
@@
 F 0 "R33" V 1280 2400 50  0000 C CNN
 F 1 "10k" V 1200 2400 50  0000 C CNN
-F 2 "Resistors_SMD:R_0805_HandSoldering" V 1130 2400 50  0001 C CNN
+F 2 "Resistor_SMD:R_0805_2012Metric_Pad1.15x1.40mm_HandSolder" V 1130 2400 50  0001 C CNN
 F 3 "" H 1200 2400 50  0000 C CNN
 	1    1200 2400
@@
 F 0 "C10" H 5125 4750 50  0000 L CNN
 F 1 "100u" H 5125 4550 50  0000 L CNN
-F 2 "Capacitors_SMD:CP_Elec_8x10" H 5100 4650 50  0001 C CNN
+F 2 "Capacitor_SMD:CP_Elec_8x10" H 5100 4650 50  0001 C CNN
 F 3 "" H 5100 4650 50  0000 C CNN
 	1    5100 4650
@@
 F 0 "C11" H 5425 4750 50  0000 L CNN
 F 1 "100u" H 5425 4550 50  0000 L CNN
-F 2 "Capacitors_SMD:CP_Elec_8x10" H 5400 4650 50  0001 C CNN
+F 2 "Capacitor_SMD:CP_Elec_8x10" H 5400 4650 50  0001 C CNN
 F 3 "" H 5400 4650 50  0000 C CNN
 	1    5400 4650
@@
 F 0 "C12" H 5725 4750 50  0000 L CNN
 F 1 "100u" H 5725 4550 50  0000 L CNN
-F 2 "Capacitors_SMD:CP_Elec_8x10" H 5700 4650 50  0001 C CNN
+F 2 "Capacitor_SMD:CP_Elec_8x10" H 5700 4650 50  0001 C CNN
 F 3 "" H 5700 4650 50  0000 C CNN
 	1    5700 4650
@@
 F 0 "C9" H 4825 4750 50  0000 L CNN
 F 1 "100u" H 4825 4550 50  0000 L CNN
-F 2 "Capacitors_SMD:CP_Elec_8x10" H 4800 4650 50  0001 C CNN
+F 2 "Capacitor_SMD:CP_Elec_8x10" H 4800 4650 50  0001 C CNN
 F 3 "" H 4800 4650 50  0000 C CNN
 	1    4800 4650
@@
 F 0 "R38" V 1430 5000 50  0000 C CNN
 F 1 "10k" V 1350 5000 50  0000 C CNN
-F 2 "Resistors_SMD:R_0805_HandSoldering" V 1280 5000 50  0001 C CNN
+F 2 "Resistor_SMD:R_0805_2012Metric_Pad1.15x1.40mm_HandSolder" V 1280 5000 50  0001 C CNN
 F 3 "" H 1350 5000 50  0000 C CNN
 	1    1350 5000
@@
 F 0 "R34" V 4130 2400 50  0000 C CNN
 F 1 "10k" V 4050 2400 50  0000 C CNN
-F 2 "Resistors_SMD:R_0805_HandSoldering" V 3980 2400 50  0001 C CNN
+F 2 "Resistor_SMD:R_0805_2012Metric_Pad1.15x1.40mm_HandSolder" V 3980 2400 50  0001 C CNN
 F 3 "" H 4050 2400 50  0000 C CNN
 	1    4050 2400
@@
 F 0 "R35" V 7230 2400 50  0000 C CNN
 F 1 "10k" V 7150 2400 50  0000 C CNN
-F 2 "Resistors_SMD:R_0805_HandSoldering" V 7080 2400 50  0001 C CNN
+F 2 "Resistor_SMD:R_0805_2012Metric_Pad1.15x1.40mm_HandSolder" V 7080 2400 50  0001 C CNN
 F 3 "" H 7150 2400 50  0000 C CNN
 	1    7150 2400
